File: unified-usb-pcb_batt/unified-usb-pcb_batt.kicad_pcb (KiCad board)
At the start: 2 copper layers, 34 parts, among them J1 QI, J2 USB_C_Receptacle_USB2.0, J3 USB_Out, J4 BATT, J5 THERM, SW1 SW_SPDT, U1 SRV05-4, U2 DW01A, U3 TP4056, U4 FS8205

Commit message: started working on pcb layout
Parts:
- moved U3 50.3 mm to (33.5, 38.6), turned to 90 degrees
- moved U4 42.6 mm to (44.0, 39.8), turned to 270 degrees
- moved J4 38.7 mm to (44.3, 28.4)
- moved U2 36.9 mm to (40.8, 45.5), turned to 180 degrees
- moved JP2 35.0 mm to (37.8, 29.5)
- moved R11 32.2 mm to (37.8, 32.3), turned to 0 degrees
- moved R8 32.0 mm to (37.8, 34.3)
- moved J5 26.9 mm to (44.3, 34.5)
- moved R9 26.8 mm to (39.5, 41.9), turned to 270 degrees
- moved J3 25.3 mm to (24.5, 44.0)
- moved R10 24.3 mm to (30.9, 43.3)
- moved C2 21.4 mm to (39.5, 38.9), turned to 0 degrees
- moved R4 20.3 mm to (37.8, 41.9)
- moved C1 19.3 mm to (37.8, 45.0), turned to 270 degrees
- moved C4 19.2 mm to (35.1, 43.3), turned to 180 degrees
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Connections:
- J4 pad 1: Net-(J4-Pad1) -> Net-(C1-Pad2)
- J4 pad 2: Net-(C1-Pad2) -> Net-(J4-Pad2)
- SW1 pad 2: Net-(J4-Pad1) -> Net-(J4-Pad2)
Routing:
- net GNDPWR: track 31.6 -> 61.0 mm, vias 3 -> 2
- net Net-(R5-Pad1): track 0.00 -> 24.2 mm, vias 0 -> 1
- net chgsense: track 1.91 -> 24.3 mm, vias 0 -> 1
- net USB_D-: track 9.27 -> 21.6 mm, vias 0 -> 1
- net USB_D+: track 9.97 -> 21.9 mm, vias 0 -> 1
- net +5V: track 24.1 -> 35.7 mm
- net Net-(J5-Pad1): track 0.00 -> 10.7 mm, vias 0 -> 1
- net VOUT: track 0.00 -> 7.72 mm
- net Net-(D1-Pad2): track 10.8 -> 14.8 mm
- net Net-(R10-Pad2): track 0.00 -> 3.96 mm
- net Net-(F2-Pad2): track 4.24 -> 5.49 mm
Other:
- board outline added: 34 x 29.2 mm

Commit message: finished pcb
Parts:
- added H1: MountingHole_Pad, MountingHole:MountingHole_2.7mm_M2.5_DIN965_Pad, F.Cu at (18.8, 21.3)
- added H2: MountingHole_Pad, MountingHole:MountingHole_2.7mm_M2.5_DIN965_Pad, F.Cu at (42.8, 21.3)
- added H3: MountingHole_Pad, MountingHole:MountingHole_2.7mm_M2.5_DIN965_Pad, F.Cu at (18.8, 50.3)
- added H4: MountingHole_Pad, MountingHole:MountingHole_2.7mm_M2.5_DIN965_Pad, F.Cu at (42.8, 50.3)
- J2: value USB_C_Receptacle_USB2.0 -> HRO C-31-M-12
- moved C4 18.4 mm to (16.8, 45.0), turned to 90 degrees
- moved C2 13.1 mm to (27.4, 43.9), turned to 90 degrees
- moved U3 13.1 mm to (21.5, 43.7), turned to 0 degrees
- moved R1 13.0 mm to (22.6, 25.7), turned to 90 degrees
- moved J4 13.0 mm to (42.4, 41.3)
- moved R10 11.7 mm to (19.7, 39.9)
- moved SW1 10.3 mm to (40.4, 34.4)
- moved R4 9.03 mm to (37.4, 50.9), turned to 0 degrees
- moved D2 8.80 mm to (26.9, 35.4)
- moved F3 8.73 mm to (23.9, 49.3), turned to 90 degrees
- moved J3 8.63 mm to (30.8, 50.0)
- moved JP1 8.53 mm to (32.2, 38.9), turned to 0 degrees
- moved C3 8.42 mm to (27.6, 38.9)
- moved D1 8.41 mm to (34.1, 35.4)
- moved F2 8.00 mm to (24.6, 31.2), turned to 90 degrees
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Routing:
- net GNDPWR: track 61.0 -> 0.57 mm
- net Net-(J5-Pad1): track 10.7 -> 52.7 mm, vias 1 -> 2
- net VOUT: track 7.72 -> 43.9 mm, vias 0 -> 1
- net +5V: track 35.7 -> 53.9 mm, vias 0 -> 5
- net chgsense: track 24.3 -> 39.5 mm, vias 1 -> 3
- net Net-(C1-Pad2): track 0.00 -> 13.5 mm
- net Net-(F3-Pad1): track 0.00 -> 9.38 mm
- net Net-(J4-Pad2): track 0.00 -> 7.43 mm, vias 0 -> 1
- net Net-(J2-PadA5): track 7.74 -> 13.2 mm
- net Net-(R5-Pad1): track 24.2 -> 29.7 mm, vias 1 -> 2
- net USB_D-: track 21.6 -> 26.9 mm, vias 1 -> 2
- net USB_D+: track 21.9 -> 26.5 mm, vias 1 -> 2
- net Net-(C1-Pad1): track 0.00 -> 4.03 mm
- net Net-(R9-Pad2): track 0.00 -> 3.89 mm
- net Net-(J2-PadS1): track 20.6 -> 24.4 mm
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- added copper zone on B.Cu, net GNDPWR
- added copper zone on F.Cu, net GNDPWR
Other:
- board size 34 x 29.2 mm -> 30 x 35 mm
- board text added: "Batt"
- board text added: "HRO C-31 M-12"
- board text added: "QI"
- board text added: "Th"
- board text added: "USB"

Commit message: added silkscreen text
Other:
- board text added: "Type-C PCB [Li-Ion] rev 1.0 github.com/ebastler/unified-usb-pcb mpwr.xyz"
Changed lines of the file:
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@@
   (general
     (thickness 1.6)
-    (drawings 13)
+    (drawings 14)
     (tracks 217)
     (zones 0)
@@
     )
   )
+  (gr_text "Type-C PCB [Li-Ion] rev 1.0\ngithub.com/ebastler/unified-usb-pcb\nmpwr.xyz" (at 45.3644 45.085) (layer B.SilkS)
+    (effects (font (size 1 1) (thickness 0.15)) (justify left mirror))
+  )
   (gr_text USB (at 32.7914 46.228) (layer F.SilkS)
