File: unified-usb-pcb_batt/unified-usb-pcb_batt.sch (KiCad schematic (older format))
At the start: 32 parts, among them J1 USB_Out, J2 USB_C_Receptacle_USB2.0, J3 QI, J4 BATT, J5 THERM, U1 SRV05-4, U2 DW01A, U3 TP4056, U4 FS8205

Commit message: added thermistor values and charge sense wire
Parts:
- added R?: 10k, Resistor_SMD:R_0603_1608Metric, symbol Device:R_Small
- R10: value 1,8k -> 22k
- R7: value 1,8k -> 3.3k
Connections:
- net labels added: chgsense
- wire segments 92 -> 100
Other:
- note added: "Internal USB header"
- moved on the sheet: C1, C2, C3, C4, D3, D4, F?, J1, J4, J5, R10, R4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

Commit message: added a jumper to disconnect battery
Parts:
- added JP?: disconnect batt, Connector_PinHeader_2.54mm:PinHeader_1x02_P2.54mm_Vertical, symbol Jumper:Jumper_2_Open
- gave numbers to parts that had none: 2
- renumbered J3 to J1, J1 to J3, R9 to R10, R10 to R11, R6 to R7, R7 to R8, R8 to R9
Connections:
- wire segments 100 -> 105
Other:
- moved on the sheet: C2
Changed lines of the file:
@@
 	1950 1300 1950 1400
 $Comp
-L power:GNDPWR #PWR02
+L power:GNDPWR #PWR04
 U 1 1 5E885EC3
 P 2150 1400
-F 0 "#PWR02" H 2150 1200 50  0001 C CNN
+F 0 "#PWR04" H 2150 1200 50  0001 C CNN
 F 1 "GNDPWR" H 2154 1246 50  0000 C CNN
 F 2 "" H 2150 1350 50  0001 C CNN
@@
 	1700 1700 2150 1700
 $Comp
-L power:GNDPWR #PWR03
+L power:GNDPWR #PWR06
 U 1 1 5E891102
 P 2850 2600
-F 0 "#PWR03" H 2850 2400 50  0001 C CNN
+F 0 "#PWR06" H 2850 2400 50  0001 C CNN
 F 1 "GNDPWR" H 2854 2446 50  0000 C CNN
 F 2 "" H 2850 2550 50  0001 C CNN
@@
 	3150 1100 3250 1100
 $Comp
-L Connector_Generic:Conn_01x05 J1
+L Connector_Generic:Conn_01x05 J3
 U 1 1 5E8A3E4C
 P 5350 2300
-F 0 "J1" H 5250 2650 50  0000 L CNN
+F 0 "J3" H 5250 2650 50  0000 L CNN
 F 1 "USB_Out" H 5150 1950 50  0000 L CNN
 F 2 "Connector_JST:JST_SH_SM05B-SRSS-TB_1x05-1MP_P1.00mm_Horizontal" H 5350 2300 50  0001 C CNN
@@
 $EndComp
 $Comp
-L Connector_Generic:Conn_01x02 J3
+L Connector_Generic:Conn_01x02 J1
 U 1 1 5E8AD69B
 P 4350 1200
-F 0 "J3" H 4400 900 50  0000 C CNN
+F 0 "J1" H 4400 900 50  0000 C CNN
 F 1 "QI" H 4400 1000 50  0000 C CNN
 F 2 "" H 4350 1200 50  0001 C CNN
@@
 $EndComp
 $Comp
-L power:GNDPWR #PWR05
+L power:GNDPWR #PWR03
 U 1 1 5E8B324F
 P 4750 1200
-F 0 "#PWR05" H 4750 1000 50  0001 C CNN
+F 0 "#PWR03" H 4750 1000 50  0001 C CNN
 F 1 "GNDPWR" H 4754 1046 50  0000 C CNN
 F 2 "" H 4750 1150 50  0001 C CNN
@@
 	4550 1100 4600 1100
 $Comp
-L power:+5V #PWR04
+L power:+5V #PWR02
 U 1 1 5E8B598D
 P 5300 1100
-F 0 "#PWR04" H 5300 950 50  0001 C CNN
+F 0 "#PWR02" H 5300 950 50  0001 C CNN
 F 1 "+5V" H 5400 1200 50  0000 C CNN
 F 2 "" H 5300 1100 50  0001 C CNN
@@
 $EndComp
 $Comp
-L Device:R_Small R6
+L Device:R_Small R7
 U 1 1 5E8CFECB
 P 1100 3900
-F 0 "R6" V 1000 4000 50  0000 C CNN
+F 0 "R7" V 1000 4000 50  0000 C CNN
 F 1 "2,7k" V 1000 3850 50  0000 C CNN
 F 2 "Resistor_SMD:R_0603_1608Metric" H 1100 3900 50  0001 C CNN
@@
 	650  4000 650  4150
 $Comp
-L Device:R_Small R9
+L Device:R_Small R10
 U 1 1 5E8D9D87
 P 2550 4250
-F 0 "R9" V 2450 4350 50  0000 C CNN
+F 0 "R10" V 2450 4350 50  0000 C CNN
 F 1 "1,8k" V 2450 4150 50  0000 C CNN
 F 2 "Resistor_SMD:R_0603_1608Metric" H 2550 4250 50  0001 C CNN
@@
 $EndComp
 $Comp
-L power:GNDPWR #PWR08
+L power:GNDPWR #PWR09
 U 1 1 5E8DAA5C
 P 2550 4450
-F 0 "#PWR08" H 2550 4250 50  0001 C CNN
+F 0 "#PWR09" H 2550 4250 50  0001 C CNN
 F 1 "GNDPWR" H 2554 4296 50  0000 C CNN
 F 2 "" H 2550 4400 50  0001 C CNN
@@
 Connection ~ 2550 4450
 $Comp
-L power:+5V #PWR06
+L power:+5V #PWR07
 U 1 1 5E8C9310
 P 1650 3500
-F 0 "#PWR06" H 1650 3350 50  0001 C CNN
+F 0 "#PWR07" H 1650 3350 50  0001 C CNN
 F 1 "+5V" H 1750 3600 50  0000 C CNN
 F 2 "" H 1650 3500 50  0001 C CNN
@@
 	3250 1100 3500 1100
 $Comp
-L Device:R_Small R7
+L Device:R_Small R8
 U 1 1 5E9144B7
 P 2800 3950
-F 0 "R7" V 2700 3950 50  0000 C CNN
+F 0 "R8" V 2700 3950 50  0000 C CNN
 F 1 "3.3k" V 2700 3800 50  0000 C CNN
 F 2 "Resistor_SMD:R_0603_1608Metric" H 2800 3950 50  0001 C CNN
@@
 $EndComp
 $Comp
-L Device:R_Small R10
+L Device:R_Small R11
 U 1 1 5E914F3C
 P 2800 4250
-F 0 "R10" V 2700 4350 50  0000 C CNN
+F 0 "R11" V 2700 4350 50  0000 C CNN
 F 1 "22k" V 2700 4150 50  0000 C CNN
 F 2 "Resistor_SMD:R_0603_1608Metric" H 2800 4250 50  0001 C CNN
@@
 Connection ~ 2800 4050
 $Comp
-L power:+5V #PWR07
+L power:+5V #PWR08
 U 1 1 5E9194DF
 P 2800 3850
-F 0 "#PWR07" H 2800 3700 50  0001 C CNN
+F 0 "#PWR08" H 2800 3700 50  0001 C CNN
 F 1 "+5V" H 2650 3950 50  0000 C CNN
 F 2 "" H 2800 3850 50  0001 C CNN
@@
 U 1 1 5E8F81D1
 P 1400 3800
-F 0 "C3" V 1250 3600 50  0000 L CNN
+F 0 "C3" V 1300 3650 50  0000 L CNN
 F 1 "10u" V 1300 3800 50  0000 L CNN
 F 2 "Capacitor_Tantalum_SMD:CP_EIA-3216-18_Kemet-A" H 1400 3800 50  0001 C CNN
@@
 	4650 3500 4750 3500
 $Comp
-L Device:R_Small R8
+L Device:R_Small R9
 U 1 1 5E98E292
 P 5350 3950
-F 0 "R8" V 5250 4050 50  0000 C CNN
+F 0 "R9" V 5250 4050 50  0000 C CNN
 F 1 "1k" V 5250 3900 50  0000 C CNN
 F 2 "Resistor_SMD:R_0603_1608Metric" H 5350 3950 50  0001 C CNN
@@
 	0    1    1    0
 $EndComp
-Connection ~ 3700 3600
 Text GLabel 3750 3350 2    50   Output ~ 0
 VOUT
@@
 L Device:CP_Small C2
 U 1 1 5E9A1A52
-P 3600 3700
-F 0 "C2" H 3350 3750 50  0000 L CNN
-F 1 "10u" H 3350 3600 50  0000 L CNN
-F 2 "Capacitor_Tantalum_SMD:CP_EIA-3216-18_Kemet-A" H 3600 3700 50  0001 C CNN
-F 3 "~" H 3600 3700 50  0001 C CNN
-	1    3600 3700
-	1    0    0    -1
-$EndComp
-Wire Wire Line
-	3200 4450 3600 4450
+P 3250 3700
+F 0 "C2" H 3000 3750 50  0000 L CNN
+F 1 "10u" H 3000 3600 50  0000 L CNN
+F 2 "Capacitor_Tantalum_SMD:CP_EIA-3216-18_Kemet-A" H 3250 3700 50  0001 C CNN
+F 3 "~" H 3250 3700 50  0001 C CNN
+	1    3250 3700
+	1    0    0    -1
+$EndComp
 Connection ~ 3200 4450
 Wire Wire Line
-	2550 3600 3600 3600
-Connection ~ 3600 3600
-Wire Wire Line
-	3600 3600 3700 3600
-Wire Wire Line
-	3600 3800 3600 4450
-Connection ~ 3600 4450
-Wire Wire Line
-	3600 4450 4250 4450
-Wire Wire Line
 	1650 3700 1800 3700
 Wire Wire Line
-	1800 3800 1800 3900
-Wire Wire Line
-	1800 3900 1650 3900
-Wire Wire Line
-	1650 3900 1650 4450
-Connection ~ 1650 3900
+	1650 3900 1650 4000
 Wire Wire Line
 	1650 4450 2550 4450
@@
 U 1 1 5EA1E00B
 P 1650 3800
-F 0 "C4" V 1550 3600 50  0000 L CNN
+F 0 "C4" V 1550 3650 50  0000 L CNN
 F 1 "100n" V 1550 3800 50  0000 L CNN
 F 2 "Capacitor_Tantalum_SMD:CP_EIA-3216-18_Kemet-A" H 1650 3800 50  0001 C CNN
@@
 	1100 4050 1800 4050
 Wire Wire Line
-	1400 3900 1650 3900
-Wire Wire Line
 	1400 3700 1650 3700
 Wire Wire Line
@@
 Wire Wire Line
 	4000 3500 3700 3500
-Connection ~ 3700 3500
-Wire Wire Line
-	3700 3500 3700 3600
 Wire Notes Line style solid
 	550  700  550  2850
@@
 $EndComp
 $Comp
-L Device:Polyfuse_Small F?
+L Device:Polyfuse_Small F3
 U 1 1 5EABBE64
 P 4850 2200
-F 0 "F?" V 4800 2350 50  0000 C CNN
+F 0 "F3" V 4800 2350 50  0000 C CNN
 F 1 "1A" V 4800 2050 50  0000 C CNN
 F 2 "" H 4900 2000 50  0001 L CNN
@@
 	4600 2400 5150 2400
 $Comp
-L power:GNDPWR #PWR?
+L power:GNDPWR #PWR05
 U 1 1 5E879D91
 P 4550 2500
-F 0 "#PWR?" H 4550 2300 50  0001 C CNN
+F 0 "#PWR05" H 4550 2300 50  0001 C CNN
 F 1 "GNDPWR" H 4554 2346 50  0000 C CNN
 F 2 "" H 4550 2450 50  0001 C CNN
@@
 	4600 2100 5150 2100
 $Comp
-L Device:R_Small R?
+L Device:R_Small R6
 U 1 1 5E89839E
 P 850 3900
-F 0 "R?" V 750 4000 50  0000 C CNN
+F 0 "R6" V 750 4000 50  0000 C CNN
 F 1 "10k" V 750 3850 50  0000 C CNN
 F 2 "Resistor_SMD:R_0603_1608Metric" H 850 3900 50  0001 C CNN
@@
 Text Notes 4150 1800 0    50   ~ 0
 Internal USB header
+Wire Wire Line
+	1400 3900 1400 4000
+Wire Wire Line
+	1400 4000 1650 4000
+Connection ~ 1650 4000
+Wire Wire Line
+	1650 4000 1650 4450
+Wire Wire Line
+	1800 4000 1650 4000
+Wire Wire Line
+	1800 3800 1800 4000
+Wire Wire Line
+	3200 4450 3650 4450
+$Comp
+L Jumper:Jumper_2_Open JP?
+U 1 1 5E8F2064
+P 3500 3600
+F 0 "JP?" H 3050 3750 50  0000 L CNN
+F 1 "disconnect batt" H 3050 3850 50  0000 L CNN
+F 2 "Connector_PinHeader_2.54mm:PinHeader_1x02_P2.54mm_Vertical" H 3500 3600 50  0001 C CNN
+F 3 "~" H 3500 3600 50  0001 C CNN
+	1    3500 3600
+	1    0    0    -1
+$EndComp
+Wire Wire Line
+	3250 3800 3250 3850
+Wire Wire Line
+	3250 3850 3650 3850
+Wire Wire Line
+	3650 3850 3650 4450
+Connection ~ 3650 4450
+Wire Wire Line
+	3650 4450 4250 4450
+Wire Wire Line
+	3700 3500 3300 3500
+Wire Wire Line
+	3300 3500 3300 3600
+Connection ~ 3700 3500
+Wire Wire Line
+	3300 3600 3250 3600
+Connection ~ 3300 3600
+Wire Wire Line
+	3250 3600 2550 3600
+Connection ~ 3250 3600
 $EndSCHEMATC

Commit message: continued with Li-Ion schematic, initialised pcb
Parts:
- C1, C4: footprint Capacitor_Tantalum_SMD:CP_EIA-3216-18_Kemet-A -> Capacitor_SMD:C_0603_1608Metric
- D1, D2: value D_Schottky -> SS34; footprint (none) -> Diode_SMD:D_SMA
- D3: value LED_GR -> 19-217/GHC-YR1S2/3T; footprint (none) -> LED_SMD:LED_0603_1608Metric_Castellated
- D4: value LED_R -> KT-0603R; footprint (none) -> LED_SMD:LED_0603_1608Metric_Castellated
- F1, F2, F3: value 1A -> 1206L050/15YR; footprint (none) -> Fuse:Fuse_1206_3216Metric
- J1, J4, J5: footprint (none) -> Connector_JST:JST_SH_SM02B-SRSS-TB_1x02-1MP_P1.00mm_Horizontal
- JP1, JP2: symbol Jumper:Jumper_2_Open -> Jumper:SolderJumper_2_Open
- JP3: renamed from JP?; symbol Jumper:Jumper_2_Open -> Jumper:Jumper_2_Bridged
Connections:
- wire segments 105 -> 107
Changed lines of the file:
@@
 $EndComp
-Wire Wire Line
-	2150 1700 2150 1650
-Wire Wire Line
-	2150 1650 2350 1650
-Wire Wire Line
-	2150 1800 2150 1850
-Wire Wire Line
-	2150 1850 2350 1850
 Wire Wire Line
 	1700 1900 1700 1800
-Connection ~ 1700 1800
 Wire Wire Line
 	1700 1600 1700 1700
-Connection ~ 1700 1700
-Wire Wire Line
-	2350 1850 2350 2300
-Wire Wire Line
-	2350 2300 3350 2300
-Wire Wire Line
-	3350 2300 3350 1850
-Connection ~ 2350 1850
-Wire Wire Line
-	2350 1650 2350 1200
-Wire Wire Line
-	2350 1200 3350 1200
-Wire Wire Line
-	3350 1200 3350 1650
-Connection ~ 2350 1650
 Wire Wire Line
 	2850 2250 2850 2600
@@
 Wire Wire Line
 	1950 1100 2850 1100
-Wire Wire Line
-	1700 1800 2150 1800
-Wire Wire Line
-	1700 1700 2150 1700
 $Comp
 L power:GNDPWR #PWR06
@@
 P 3000 1100
 F 0 "D1" H 2850 1050 50  0000 C CNN
-F 1 "D_Schottky" H 2700 1150 50  0000 C CNN
-F 2 "" H 3000 1100 50  0001 C CNN
+F 1 "SS34" H 2700 1150 50  0000 C CNN
+F 2 "Diode_SMD:D_SMA" H 3000 1100 50  0001 C CNN
 F 3 "https://datasheet.lcsc.com/szlcsc/Vishay-Intertech-SS36-E3-57T_C35722.pdf" H 3000 1100 50  0001 C CNN
 	1    3000 1100
@@
 F 0 "J4" H 3980 3592 50  0000 L CNN
 F 1 "BATT" H 3980 3501 50  0000 L CNN
-F 2 "" H 3900 3600 50  0001 C CNN
+F 2 "Connector_JST:JST_SH_SM02B-SRSS-TB_1x02-1MP_P1.00mm_Horizontal" H 3900 3600 50  0001 C CNN
 F 3 "~" H 3900 3600 50  0001 C CNN
 	1    3900 3600
@@
 F 0 "J5" H 3480 4042 50  0000 L CNN
 F 1 "THERM" H 3250 3850 50  0000 L CNN
-F 2 "" H 3400 4050 50  0001 C CNN
+F 2 "Connector_JST:JST_SH_SM02B-SRSS-TB_1x02-1MP_P1.00mm_Horizontal" H 3400 4050 50  0001 C CNN
 F 3 "~" H 3400 4050 50  0001 C CNN
 	1    3400 4050
@@
 F 0 "J1" H 4400 900 50  0000 C CNN
 F 1 "QI" H 4400 1000 50  0000 C CNN
-F 2 "" H 4350 1200 50  0001 C CNN
+F 2 "Connector_JST:JST_SH_SM02B-SRSS-TB_1x02-1MP_P1.00mm_Horizontal" H 4350 1200 50  0001 C CNN
 F 3 "~" H 4350 1200 50  0001 C CNN
 	1    4350 1200
@@
 P 5000 1100
 F 0 "D2" H 5000 884 50  0000 C CNN
-F 1 "D_Schottky" H 5000 975 50  0000 C CNN
-F 2 "" H 5000 1100 50  0001 C CNN
+F 1 "SS34" H 5000 975 50  0000 C CNN
+F 2 "Diode_SMD:D_SMA" H 5000 1100 50  0001 C CNN
 F 3 "https://datasheet.lcsc.com/szlcsc/Vishay-Intertech-SS36-E3-57T_C35722.pdf" H 5000 1100 50  0001 C CNN
 	1    5000 1100
@@
 P 4700 1100
 F 0 "F2" V 4500 1000 50  0000 C CNN
-F 1 "1A" V 4600 1000 50  0000 C CNN
-F 2 "" H 4750 900 50  0001 L CNN
+F 1 "1206L050/15YR" V 4400 1000 50  0000 C CNN
+F 2 "Fuse:Fuse_1206_3216Metric" H 4750 900 50  0001 L CNN
 F 3 "https://datasheet.lcsc.com/szlcsc/1810252220_Fuzetec-Tech-FSMD050-1206-R_C220147.pdf" H 4700 1100 50  0001 C CNN
 	1    4700 1100
@@
 P 650 3700
 F 0 "D3" H 700 3600 50  0000 R CNN
-F 1 "LED_GR" V 900 3700 50  0000 R CNN
-F 2 "" V 650 3700 50  0001 C CNN
+F 1 "19-217/GHC-YR1S2/3T" V 900 3700 50  0000 R CNN
+F 2 "LED_SMD:LED_0603_1608Metric_Castellated" V 650 3700 50  0001 C CNN
 F 3 "~" V 650 3700 50  0001 C CNN
 	1    650  3700
@@
 P 1100 3700
 F 0 "D4" H 1150 3600 50  0000 R CNN
-F 1 "LED_R" V 1250 3900 50  0000 R CNN
-F 2 "" V 1100 3700 50  0001 C CNN
+F 1 "KT-0603R" V 1250 3900 50  0000 R CNN
+F 2 "LED_SMD:LED_0603_1608Metric_Castellated" V 1100 3700 50  0001 C CNN
 F 3 "~" V 1100 3700 50  0001 C CNN
 	1    1100 3700
@@
 $EndComp
 $Comp
-L Jumper:Jumper_2_Open JP2
+L Jumper:SolderJumper_2_Open JP2
 U 1 1 5E8EA6C4
 P 3000 4250
@@
 	1    0    0    -1
 $EndComp
-Wire Wire Line
-	3350 1650 3400 1650
-Connection ~ 3350 1650
-Wire Wire Line
-	3350 1850 3400 1850
-Connection ~ 3350 1850
-$Comp
-L Jumper:Jumper_2_Open JP1
+$Comp
+L Jumper:SolderJumper_2_Open JP1
 U 1 1 5E906293
 P 3050 900
@@
 Wire Wire Line
 	2800 4150 2800 4050
-Wire Wire Line
-	2800 4050 3000 4050
 Connection ~ 2800 4050
 $Comp
@@
 Connection ~ 3000 4450
 Wire Wire Line
-	3200 4050 3000 4050
-Connection ~ 3000 4050
-Wire Wire Line
 	3700 3700 3700 3850
 Wire Wire Line
@@
 F 0 "C1" H 4350 3600 50  0000 L CNN
 F 1 "100n" H 4350 3500 50  0000 L CNN
-F 2 "Capacitor_Tantalum_SMD:CP_EIA-3216-18_Kemet-A" H 4650 3600 50  0001 C CNN
+F 2 "Capacitor_SMD:C_0603_1608Metric" H 4650 3600 50  0001 C CNN
 F 3 "~" H 4650 3600 50  0001 C CNN
 	1    4650 3600
@@
 F 0 "C4" V 1550 3650 50  0000 L CNN
 F 1 "100n" V 1550 3800 50  0000 L CNN
-F 2 "Capacitor_Tantalum_SMD:CP_EIA-3216-18_Kemet-A" H 1650 3800 50  0001 C CNN
+F 2 "Capacitor_SMD:C_0603_1608Metric" H 1650 3800 50  0001 C CNN
 F 3 "~" H 1650 3800 50  0001 C CNN
 	1    1650 3800
@@
 P 1850 1100
 F 0 "F1" V 1750 1200 50  0000 C CNN
-F 1 "1A" V 1750 1000 50  0000 C CNN
-F 2 "" H 1900 900 50  0001 L CNN
+F 1 "1206L050/15YR" V 1650 1350 50  0000 C CNN
+F 2 "Fuse:Fuse_1206_3216Metric" H 1900 900 50  0001 L CNN
 F 3 "https://datasheet.lcsc.com/szlcsc/1810252220_Fuzetec-Tech-FSMD050-1206-R_C220147.pdf" H 1850 1100 50  0001 C CNN
 	1    1850 1100
@@
 P 4850 2200
 F 0 "F3" V 4800 2350 50  0000 C CNN
-F 1 "1A" V 4800 2050 50  0000 C CNN
-F 2 "" H 4900 2000 50  0001 L CNN
+F 1 "1206L050/15YR" V 4600 2200 50  0000 C CNN
+F 2 "Fuse:Fuse_1206_3216Metric" H 4900 2000 50  0001 L CNN
 F 3 "https://datasheet.lcsc.com/szlcsc/1810252220_Fuzetec-Tech-FSMD050-1206-R_C220147.pdf" H 4850 2200 50  0001 C CNN
 	1    4850 2200
@@
 	3200 4450 3650 4450
 $Comp
-L Jumper:Jumper_2_Open JP?
+L Jumper:Jumper_2_Bridged JP3
 U 1 1 5E8F2064
 P 3500 3600
-F 0 "JP?" H 3050 3750 50  0000 L CNN
+F 0 "JP3" H 3050 3750 50  0000 L CNN
 F 1 "disconnect batt" H 3050 3850 50  0000 L CNN
 F 2 "Connector_PinHeader_2.54mm:PinHeader_1x02_P2.54mm_Vertical" H 3500 3600 50  0001 C CNN
@@
 	3250 3600 2550 3600
 Connection ~ 3250 3600
+Wire Wire Line
+	3000 4400 3000 4450
+Wire Wire Line
+	2800 4050 3000 4050
+Wire Wire Line
+	3000 4100 3000 4050
+Connection ~ 3000 4050
+Wire Wire Line
+	3000 4050 3200 4050
+Wire Wire Line
+	2900 900  2850 900
+Wire Wire Line
+	3200 900  3250 900
+Wire Wire Line
+	3350 1650 3350 1850
+Wire Wire Line
+	2350 1650 2350 1850
+Wire Wire Line
+	3400 1650 3350 1650
+Connection ~ 3350 1650
+Wire Wire Line
+	3350 1650 3350 1200
+Wire Wire Line
+	3350 1200 2300 1200
+Wire Wire Line
+	2300 1200 2300 1600
+Wire Wire Line
+	2300 1600 1700 1600
+Connection ~ 1700 1600
+Wire Wire Line
+	1700 1900 2350 1900
+Wire Wire Line
+	2350 1900 2350 1850
+Connection ~ 1700 1900
+Connection ~ 2350 1850
+Wire Wire Line
+	2350 1900 2350 2300
+Wire Wire Line
+	2350 2300 3400 2300
+Wire Wire Line
+	3400 2300 3400 1850
+Connection ~ 2350 1900
 $EndSCHEMATC
